File: schematics/STM32F0.kicad_sch (KiCad schematic)
At the start: 21 parts, among them J2 Conn_ARM_SWD_TagConnect_TC203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, Q1 2N7002, SW13 SW_Push, U1 STM32F072CBTx, Y1 8MHz

Commit message: Add crystal to lib, update stm link
Parts:
- Y1: footprint LocalLib:Crystal_SMD_ECX-32-4Pin_3.2x2.5mm -> Mad_Footprints:Crystal_SMD_ECX-32-4Pin_3.2x2.5mm
Changed lines of the file:
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@@
 			)
 		)
-		(property "Footprint" "LocalLib:Crystal_SMD_ECX-32-4Pin_3.2x2.5mm"
+		(property "Footprint" "Mad_Footprints:Crystal_SMD_ECX-32-4Pin_3.2x2.5mm"
 			(at 85.09 90.805 0)
 			(effects
