File: schematics/Keyboard Controllers/Controller_RP2040.kicad_sch (KiCad schematic)
At the start: 9 parts, among them J2 Conn_ARM_SWD_TagConnect_TC203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, U3 NCP1117-3.3_SOT223

Commit message: add todo
Connections:
- net 3V3: no longer D2.1 (K)
- net VBUS: no longer names the net of R3.1
Other:
- note added: "Update"
Changed lines of the file:
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@@
 	(wire
 		(pts
-			(xy 199.39 84.455) (xy 199.39 86.995)
+			(xy 199.39 83.185) (xy 199.39 85.725)
 		)
 		(stroke
@@
 			(width 0)
 			(type solid)
+		)
+	)
+	(wire
+		(pts
+			(xy 191.77 83.185) (xy 199.39 83.185)
+		)
+		(stroke
+			(width 0)
+			(type default)
 		)
 	)
@@
 		)
 	)
+	(text "Update"
+		(exclude_from_sim no)
+		(at 268.605 33.02 0)
+		(effects
+			(font
+				(size 2 2)
+				(thickness 0.4)
+				(bold yes)
+			)
+		)
+	)
 	(text "Power LED"
 		(exclude_from_sim no)
@@
 	)
 	(label "3V3"
-		(at 262.89 46.355 0)
+		(at 191.77 83.185 0)
 		(fields_autoplaced yes)
 		(effects
@@
 					(unit 1)
 				)
-			)
-		)
-	)
-	(symbol
-		(lib_id "power:VBUS")
-		(at 199.39 84.455 0)
-		(unit 1)
-		(exclude_from_sim no)
-		(in_bom yes)
-		(on_board yes)
-		(dnp no)
-		(property "Reference" "#PWR06"
-			(at 199.39 88.265 0)
-			(effects
-				(font
-					(size 1.27 1.27)
-				)
-				(hide yes)
-			)
-		)
-		(property "Value" "VBUS"
-			(at 199.39 80.01 0)
-			(effects
-				(font
-					(size 1.27 1.27)
-				)
-			)
-		)
-		(property "Footprint" ""
-			(at 199.39 84.455 0)
-			(effects
-				(font
-					(size 1.27 1.27)
-				)
-				(hide yes)
-			)
-		)
-		(property "Datasheet" ""
-			(at 199.39 84.455 0)
-			(effects
-				(font
-					(size 1.27 1.27)
-				)
-				(hide yes)
-			)
-		)
-		(property "Description" "Power symbol creates a global label with name \"VBUS\""
-			(at 199.39 84.455 0)
-			(effects
-				(font
-					(size 1.27 1.27)
-				)
-				(hide yes)
-			)
-		)
-		(pin "1"
-		)
-		(instances
-			(project "Controller_RP2040"
-				(path "/ba62e47e-9e07-4e97-ab08-24b670d50f97"
-					(reference "#PWR06")
-					(unit 1)
-				)
-			)
-			(project "Mad_RP2040"
-				(path "/eedae293-eb5b-47bd-b383-bccfdf81bf72/4e3cb99d-3a42-46ca-abb7-444fcb451820"
-					(reference "#PWR06")
-					(unit 1)
-				)

Commit message: Update schematic
Connections:
- net 3V3: now also R3.1
- net GND: now also D2.1 (K)
Changed lines of the file:
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@@
 	(wire
 		(pts
-			(xy 199.39 83.185) (xy 199.39 85.725)
+			(xy 199.39 83.185) (xy 199.39 86.995)
 		)
 		(stroke
@@
 			)
 			(justify right bottom)
+		)
+	)
+	(label "GND"
+		(at 262.89 46.355 0)
+		(fields_autoplaced yes)
+		(effects
+			(font
+				(size 1.27 1.27)
+			)
+			(justify left bottom)
 		)
 	)
@@
 				)
 			)
-			(project "Mad_RP2040"
-				(path "/eedae293-eb5b-47bd-b383-bccfdf81bf72/4e3cb99d-3a42-46ca-abb7-444fcb451820"
+			(project "CrumbCatcherLight"
+				(path "/eedae293-eb5b-47bd-b383-bccfdf81bf72/d6e61d54-5c6d-43d3-8cde-aaa69c4aea8b"
 					(reference "R15")
 					(unit 1)
@@
 				)
 			)
-			(project "Mad_RP2040"
-				(path "/eedae293-eb5b-47bd-b383-bccfdf81bf72/4e3cb99d-3a42-46ca-abb7-444fcb451820"
+			(project "CrumbCatcherLight"
+				(path "/eedae293-eb5b-47bd-b383-bccfdf81bf72/d6e61d54-5c6d-43d3-8cde-aaa69c4aea8b"
 					(reference "D2")
 					(unit 1)
@@
 				)
 			)
-			(project "Mad_RP2040"
-				(path "/eedae293-eb5b-47bd-b383-bccfdf81bf72/4e3cb99d-3a42-46ca-abb7-444fcb451820"
+			(project "CrumbCatcherLight"
+				(path "/eedae293-eb5b-47bd-b383-bccfdf81bf72/d6e61d54-5c6d-43d3-8cde-aaa69c4aea8b"
 					(reference "U3")
 					(unit 1)
@@
 				)
 			)
-			(project "Mad_RP2040"
-				(path "/eedae293-eb5b-47bd-b383-bccfdf81bf72/4e3cb99d-3a42-46ca-abb7-444fcb451820"
+			(project "CrumbCatcherLight"
+				(path "/eedae293-eb5b-47bd-b383-bccfdf81bf72/d6e61d54-5c6d-43d3-8cde-aaa69c4aea8b"
 					(reference "J2")
 					(unit 1)
@@
 				)
 			)
-			(project "Mad_RP2040"
-				(path "/eedae293-eb5b-47bd-b383-bccfdf81bf72/4e3cb99d-3a42-46ca-abb7-444fcb451820"
+			(project "CrumbCatcherLight"
+				(path "/eedae293-eb5b-47bd-b383-bccfdf81bf72/d6e61d54-5c6d-43d3-8cde-aaa69c4aea8b"
 					(reference "R4")
 					(unit 1)
@@
 				)
 			)
-			(project "Mad_RP2040"
-				(path "/eedae293-eb5b-47bd-b383-bccfdf81bf72/4e3cb99d-3a42-46ca-abb7-444fcb451820"
+			(project "CrumbCatcherLight"
+				(path "/eedae293-eb5b-47bd-b383-bccfdf81bf72/d6e61d54-5c6d-43d3-8cde-aaa69c4aea8b"
 					(reference "C4")
 					(unit 1)
@@
 				)
 			)
-			(project "Mad_RP2040"
-				(path "/eedae293-eb5b-47bd-b383-bccfdf81bf72/4e3cb99d-3a42-46ca-abb7-444fcb451820"
+			(project "CrumbCatcherLight"
+				(path "/eedae293-eb5b-47bd-b383-bccfdf81bf72/d6e61d54-5c6d-43d3-8cde-aaa69c4aea8b"
 					(reference "D1")
 					(unit 1)
@@
 				)
 			)
-			(project "Mad_RP2040"
-				(path "/eedae293-eb5b-47bd-b383-bccfdf81bf72/4e3cb99d-3a42-46ca-abb7-444fcb451820"
+			(project "CrumbCatcherLight"
+				(path "/eedae293-eb5b-47bd-b383-bccfdf81bf72/d6e61d54-5c6d-43d3-8cde-aaa69c4aea8b"
 					(reference "R3")
 					(unit 1)
@@
 				)
 			)
-			(project "Mad_RP2040"
-				(path "/eedae293-eb5b-47bd-b383-bccfdf81bf72/4e3cb99d-3a42-46ca-abb7-444fcb451820"
+			(project "CrumbCatcherLight"
+				(path "/eedae293-eb5b-47bd-b383-bccfdf81bf72/d6e61d54-5c6d-43d3-8cde-aaa69c4aea8b"
 					(reference "C5")
 					(unit 1)
@@
 		)
 		(instances
-			(project "Mad_RP2040"
-				(path "/eedae293-eb5b-47bd-b383-bccfdf81bf72/4e3cb99d-3a42-46ca-abb7-444fcb451820"
-					(page "4")
-				)
-			)
 			(project "Controller_RP2040"
 				(path "/ba62e47e-9e07-4e97-ab08-24b670d50f97"
@@
 				)
 			)
-		)
-	)
-	(sheet_instances
-		(path "/"
-			(page "1")
-		)
-	)
+			(project "CrumbCatcherLight"
+				(path "/eedae293-eb5b-47bd-b383-bccfdf81bf72/d6e61d54-5c6d-43d3-8cde-aaa69c4aea8b"
+					(page "2")
+				)
+			)
+		)
+	)

Commit message: Cleanup design blocks, add bq240xx
Parts:
- C4, C5: LCSC (none) -> C2932476; Supplier PN 311-1869-1-ND -> (none); digikey (none) -> 311-1869-1-ND; mouser (none) -> 603-CC805KKX5R8BB106
- U3: value NCP1117-3.3_SOT223 -> NCP1117-3.3; LCSC (none) -> C146799; MPN NCP1117LPSTADT3G -> NCP1117LPST33T3G; Supplier PN NCP1117LPSTADT3GOSCT-ND -> (none); digikey (none) -> NCP1117LPST33T3GOSCT-ND; mouser (none) -> 863-NCP1117LPST33T3G

Commit message: Update lib, embed models into footprints and remove from models folder
Parts:
- C4, C5: Supplier PN (none) -> 311-1869-1-ND
- D1: MPN  WS2812C-2020 -> (none); Manufacturer Worldsemi -> Worldsemi
- R15, R3, R4: Price $0.16 -> $0.16
Changed lines of the file:
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@@
 			)
 		)
-		(property "Price" "$0.16 "
+		(property "Price" "$0.16"
 			(at 269.875 33.02 0)
 			(effects
@@
 			)
 		)
-		(property "Price" "$0.16 "
+		(property "Price" "$0.16"
 			(at 199.39 99.695 0)
 			(effects
@@
 			)
 		)
-		(property "Supplier PN" ""
+		(property "Supplier PN" "311-1869-1-ND"
 			(at 53.34 64.135 0)
 			(effects
@@
 			)
 		)
-		(property "MPN " "WS2812C-2020"
-			(at 235.585 32.385 0)
-			(effects
-				(font
-					(size 1.27 1.27)
-				)
-				(hide yes)
-			)
-		)
-		(property "Manufacturer" "Worldsemi "
+		(property "Manufacturer" "Worldsemi"
 			(at 235.585 32.385 0)
 			(effects
@@
 		)
 		(property "MPN" "WS2812B-2020 "
+			(at 235.585 32.385 0)
+			(effects
+				(font
+					(size 1.27 1.27)
+				)
+				(hide yes)
+			)
+		)
+		(property "LCSC" ""
+			(at 235.585 32.385 0)
+			(effects
+				(font
+					(size 1.27 1.27)
+				)
+				(hide yes)
+			)
+		)
+		(property "Config" ""
+			(at 235.585 32.385 0)
+			(effects
+				(font
+					(size 1.27 1.27)
+				)
+				(hide yes)
+			)
+		)
+		(property "digikey" ""
+			(at 235.585 32.385 0)
+			(effects
+				(font
+					(size 1.27 1.27)
+				)
+				(hide yes)
+			)
+		)
+		(property "mouser" ""
 			(at 235.585 32.385 0)
 			(effects
@@
 			)
 		)
-		(property "Price" "$0.16 "
+		(property "Price" "$0.16"
 			(at 199.39 89.535 0)
 			(effects
@@
 			)
 		)
-		(property "Supplier PN" ""
+		(property "Supplier PN" "311-1869-1-ND"
 			(at 80.645 64.135 0)
 			(effects
